Commit message: 4 point contact added

File: src/robot_description/urdf/robot.xacro (robot description, xacro)
@@ -36,6 +36,52 @@
             <material name="blue"/>
         </visual>
+        <!-- caster front -->
+        <collision name="caster_front_collision">
+            <origin rpy=" 0 0 0" xyz="0.25 0 -0.05"/>
+            <geometry>
+              <sphere radius="0.05"/>
+            </geometry>
+            <surface>
+              <friction>
+                <ode>
+                  <mu>0</mu>
+                  <mu2>0</mu2>
+                  <slip1>1.0</slip1>
+                  <slip2>1.0</slip2>
+                </ode>
+              </friction>
+            </surface>
+        </collision>
+        <visual name="caster_front_visual">
+            <origin rpy=" 0 0 0" xyz="0.2 0 -0.05"/>
+            <geometry>
+              <sphere radius="0.05"/>
+            </geometry>
+        </visual>
+        <!-- caster back -->
+        <collision name="caster_back_collision">
+          <origin rpy=" 0 0 0" xyz="-0.25 0 -0.05"/>
+          <geometry>
+            <sphere radius="0.05"/>
+          </geometry>
+          <surface>
+            <friction>
+              <ode>
+                <mu>0</mu>
+                <mu2>0</mu2>
+                <slip1>1.0</slip1>
+                <slip2>1.0</slip2>
+              </ode>
+            </friction>
+          </surface>
+        </collision>
+        <visual name="caster_back_visual">
+          <origin rpy=" 0 0 0" xyz="-0.2 0 -0.05"/>
+          <geometry>
+            <sphere radius="0.05"/>
+          </geometry>
+        </visual>
     </link>
-  <!-- Create wheel right -->
+<!-- Create wheel right -->
   <link name="link_right_wheel">
     <inertial>
@@ -59,5 +105,5 @@
   <!--   Joint for right wheel  -->
   <joint name="joint_right_wheel" type="continuous">
-    <origin rpy="0 0 0" xyz="0 0.29 0"/>
+    <origin rpy="0 0 0" xyz="0 0.3 0"/>
     <child link="link_right_wheel" />
     <parent link="link_chassis"/>
@@ -86,7 +132,7 @@
     </visual>
   </link>
-  <!--   Joint for right wheel  -->
+  <!--   Joint for left wheel  -->
   <joint name="joint_left_wheel" type="continuous">
-    <origin rpy="0 0 0" xyz="0 -0.29 0"/>
+    <origin rpy="0 0 0" xyz="0 -0.3 0"/>
     <child link="link_left_wheel" />
     <parent link="link_chassis"/>
@@ -95,3 +141,18 @@
     <joint_properties damping="1.0" friction="1.0" />
   </joint>
+  <gazebo>
+      <plugin filename="libgazebo_ros_diff_drive.so" name="differential_drive_controller">
+        <alwaysOn>true</alwaysOn>
+        <updateRate>20</updateRate>
+        <leftJoint>joint_left_wheel</leftJoint>
+        <rightJoint>joint_right_wheel</rightJoint>
+        <wheelSeparation>0.4</wheelSeparation>
+        <wheelDiameter>0.2</wheelDiameter>
+        <torque>0.1</torque>
+        <commandTopic>cmd_vel</commandTopic>
+        <odometryTopic>odom</odometryTopic>
+        <odometryFrame>odom</odometryFrame>
+        <robotBaseFrame>link_chassis</robotBaseFrame>
+      </plugin>
+  </gazebo>
 </robot>

Commit message: Laser Sensor Added

File: src/robot_description/urdf/robot.xacro (robot description, xacro)
@@ -1,30 +1,22 @@
 <?xml version="1.0"?>
 <robot name="WRO" xmlns:xacro="https://www.ros.org/wiki/xacro" >
-    <material name="blue">
-        <color rgba="0.203125 0.23828125 0.28515625 1.0"/>
-     </material>
-     <material name="orange">
-        <color rgba="1.0 0.423529411765 0.0392156862745 1.0"/>
-    </material>
-    <gazebo reference="link_chassis">
-        <material>Gazebo/Orange</material>
-    </gazebo>
-    <gazebo reference="link_left_wheel">
-        <material>Gazebo/Blue</material>
-    </gazebo>
-    <gazebo reference="link_right_wheel">
-        <material>Gazebo/Blue</material>
-    </gazebo>
+    <xacro:include filename="$(find robot_description)/urdf/materials.xacro" />
+    <xacro:include filename="$(find robot_description)/urdf/robot.gazebo" />
+    <xacro:include filename="$(find robot_description)/urdf/macro.xacro" />
     <!-- 1st Link-->>
     <link name="link_chassis">
         <pose>0 0 0.1 0 0 0</pose>
         <inertial>
-            <mass value="5"/>
+            <!--inertia ixx="${mass*(3*r*r+l*l)/12}" ixy = "0" ixz = "0"
+                        iyy="${mass*(3*r*r+l*l)/12}" iyz = "0" izz="${mass*(r*r)/2}" /-->
+            <mass value="10"/>
             <origin rpy="0 0 0" xyz="0 0 0.1"/>
-            <inertia ixx="0.0395416666667" ixy="0" ixz="0" iyy="0.106208333333" iyz="0" izz="0.106208333333"/>
+            <inertia ixx="0.2290833333" ixy = "0" ixz = "0"
+                    iyy="0.2290833333" iyz = "0"
+                    izz="0.45" />
         </inertial>
         <collision name="collision_chassis">
             <geometry>
-                <cylinder length="0.10" radius="0.3"/>
+                <cylinder length="0.07" radius="0.3"/>
             </geometry>
         </collision>
@@ -32,34 +24,11 @@
             <origin rpy="0 0 0" xyz="0 0 0"/>
             <geometry>
-                <cylinder length="0.10" radius="0.3"/>
+                <cylinder length="0.07" radius="0.3"/>
             </geometry>
             <material name="blue"/>
         </visual>
-        <!-- caster front -->
+    <!-- caster front -->
         <collision name="caster_front_collision">
-            <origin rpy=" 0 0 0" xyz="0.25 0 -0.05"/>
-            <geometry>
-              <sphere radius="0.05"/>
-            </geometry>
-            <surface>
-              <friction>
-                <ode>
-                  <mu>0</mu>
-                  <mu2>0</mu2>
-                  <slip1>1.0</slip1>
-                  <slip2>1.0</slip2>
-                </ode>
-              </friction>
-            </surface>
-        </collision>
-        <visual name="caster_front_visual">
-            <origin rpy=" 0 0 0" xyz="0.2 0 -0.05"/>
-            <geometry>
-              <sphere radius="0.05"/>
-            </geometry>
-        </visual>
-        <!-- caster back -->
-        <collision name="caster_back_collision">
-          <origin rpy=" 0 0 0" xyz="-0.25 0 -0.05"/>
+          <origin rpy=" 0 0 0" xyz="0.30 0 -0.05"/>
           <geometry>
             <sphere radius="0.05"/>
@@ -76,6 +45,6 @@
           </surface>
         </collision>
-        <visual name="caster_back_visual">
-          <origin rpy=" 0 0 0" xyz="-0.2 0 -0.05"/>
+        <visual name="caster_front_visual">
+          <origin rpy=" 0 0 0" xyz="0.2 0 -0.05"/>
           <geometry>
             <sphere radius="0.05"/>
@@ -83,76 +52,36 @@
         </visual>
     </link>
-<!-- Create wheel right -->
-  <link name="link_right_wheel">
+ <link name="sensor_laser">
     <inertial>
-      <mass value="0.2"/>
-      <origin rpy="0 1.5707 1.5707" xyz="0 0 0"/>
-      <inertia ixx="0.00052666666" ixy="0" ixz="0" iyy="0.00052666666" iyz="0" izz="0.001"/>
+      <origin xyz="0 0 0" rpy="0 0 0" />
+      <mass value="1" />
+      <inertia ixx="0.001458333333" ixy="0" ixz="0"
+       iyy="0.001458333333" iyz="0"
+        izz="0.00125"/>
     </inertial>
-    <collision name="link_right_wheel_collision">
-      <origin rpy="0 1.5707 1.5707" xyz="0 0 0" />
+    <visual>
+      <origin xyz="0 0 0" rpy="0 0 0" />
       <geometry>
-        <cylinder length="0.04" radius="0.1"/>
+        <cylinder radius="0.05" length="0.1"/>
+      </geometry>
+      <material name="white" />
+    </visual>
+    <collision>
+      <origin xyz="0 0 0" rpy="0 0 0"/>
+      <geometry>
+        <cylinder radius="0.05" length="0.1"/>
       </geometry>
     </collision>
-    <visual name="link_right_wheel_visual">
-      <origin rpy="0 1.5707 1.5707" xyz="0 0 0"/>
-      <geometry>
-        <cylinder length="0.04" radius="0.1"/>
-      </geometry>
-    </visual>
   </link>
-  <!--   Joint for right wheel  -->
-  <joint name="joint_right_wheel" type="continuous">
-    <origin rpy="0 0 0" xyz="0 0.3 0"/>
-    <child link="link_right_wheel" />
+  <joint name="joint_sensor_laser" type="fixed">
+    <origin xyz="0.23 0 0.05" rpy="0 0 0"/>
     <parent link="link_chassis"/>
-    <axis rpy="0 0 0" xyz="0 1 0"/>
-    <limit effort="10000" velocity="1000"/>
-    <joint_properties damping="1.0" friction="1.0" />
+    <child link="sensor_laser"/>
   </joint>
-  <!-- Left Wheel link -->
-  <link name="link_left_wheel">
-    <inertial>
-      <mass value="0.2"/>
-      <origin rpy="0 1.5707 1.5707" xyz="0 0 0"/>
-      <inertia ixx="0.00052666666" ixy="0" ixz="0" iyy="0.00052666666" iyz="0" izz="0.001"/>
-    </inertial>
-    <collision name="link_left_wheel_collision">
-      <origin rpy="0 1.5707 1.5707" xyz="0 0 0" />
-      <geometry>
-        <cylinder length="0.04" radius="0.1"/>
-      </geometry>
-    </collision>
-    <visual name="link_left_wheel_visual">
-      <origin rpy="0 1.5707 1.5707" xyz="0 0 0"/>
-      <geometry>
-        <cylinder length="0.04" radius="0.1"/>
-      </geometry>
-    </visual>
-  </link>
-  <!--   Joint for left wheel  -->
-  <joint name="joint_left_wheel" type="continuous">
-    <origin rpy="0 0 0" xyz="0 -0.3 0"/>
-    <child link="link_left_wheel" />
-    <parent link="link_chassis"/>
-    <axis rpy="0 0 0" xyz="0 1 0"/>
-    <limit effort="10000" velocity="1000"/>
-    <joint_properties damping="1.0" friction="1.0" />
-  </joint>
-  <gazebo>
-      <plugin filename="libgazebo_ros_diff_drive.so" name="differential_drive_controller">
-        <alwaysOn>true</alwaysOn>
-        <updateRate>20</updateRate>
-        <leftJoint>joint_left_wheel</leftJoint>
-        <rightJoint>joint_right_wheel</rightJoint>
-        <wheelSeparation>0.4</wheelSeparation>
-        <wheelDiameter>0.2</wheelDiameter>
-        <torque>0.1</torque>
-        <commandTopic>cmd_vel</commandTopic>
-        <odometryTopic>odom</odometryTopic>
-        <odometryFrame>odom</odometryFrame>
-        <robotBaseFrame>link_chassis</robotBaseFrame>
-      </plugin>
-  </gazebo>
+  <!-- Create right wheel -->
+  <xacro:link_wheel name="link_right_wheel" />
+  <xacro:joint_wheel name="joint_right_wheel"  child="link_right_wheel"  origin_xyz="-0.05 0.28 0"  />
+	 <!-- Create left wheel -->
+  <xacro:link_wheel name="link_left_wheel" />
+  <xacro:joint_wheel name="joint_left_wheel"   child="link_left_wheel"   origin_xyz="-0.05 -0.28 0"  />
 </robot>
