Commit message: Satisfied with navigation

File: src/robot_description/urdf/macro.xacro (robot description, xacro)
@@ -11,5 +11,5 @@
               <origin rpy="0 1.5707 1.5707" xyz="0 0 0"/>
               <geometry>
-                <cylinder length="0.05" radius="0.1"/>
+                <cylinder length="0.04" radius="0.1"/>
               </geometry>
             </collision>
@@ -17,5 +17,5 @@
               <origin rpy="0 1.5707 1.5707" xyz="0 0 0"/>
               <geometry>
-                <cylinder length="0.05" radius="0.1"/>
+                <cylinder length="0.04" radius="0.1"/>
               </geometry>
             </visual>
@@ -32,3 +32,34 @@
       </joint>
     </xacro:macro>
+    <xacro:macro name="link_sensor" params="name">
+       <link name="${name}">
+        <inertial>
+          <origin xyz="0 0 0" rpy="0 0 0" />
+          <mass value="1" />
+          <inertia ixx="0.001458333333" ixy="0" ixz="0"
+          iyy="0.001458333333" iyz="0"
+          izz="0.00125"/>
+        </inertial>
+        <visual>
+          <origin xyz="0 0 0" rpy="0 0 0" />
+          <geometry>
+            <cylinder radius="0.05" length="0.1"/>
+          </geometry>
+          <material name="white" />
+        </visual>
+        <collision>
+          <origin xyz="0 0 0" rpy="0 0 0"/>
+          <geometry>
+            <cylinder radius="0.05" length="0.1"/>
+          </geometry>
+        </collision>
+      </link>
+    </xacro:macro>
+    <xacro:macro name="joint_Sensor" params="name child ">
+      <joint name="joint_sensor_laser" type="fixed">
+        <origin xyz="0.25 0 0.05" rpy="0 0 0"/>
+        <parent link="link_chassis"/>
+        <child link="${child}"/>
+      </joint>
+    </xacro:macro>
 </robot>

File: src/robot_description/urdf/robot.xacro (robot description, xacro)
@@ -10,9 +10,9 @@
             <!--inertia ixx="${mass*(3*r*r+l*l)/12}" ixy = "0" ixz = "0"
                         iyy="${mass*(3*r*r+l*l)/12}" iyz = "0" izz="${mass*(r*r)/2}" /-->
-            <mass value="10"/>
+            <mass value="15"/>
             <origin rpy="0 0 0" xyz="0 0 0.1"/>
             <inertia ixx="0.2290833333" ixy = "0" ixz = "0"
-                    iyy="0.2290833333" iyz = "0"
-                    izz="0.45" />
+                     iyy="0.2290833333" iyz = "0"
+                     izz="0.45" />
         </inertial>
         <collision name="collision_chassis">
@@ -28,7 +28,16 @@
             <material name="blue"/>
         </visual>
+    </link>
+    <link name="link_caster">
+        <inertial>
+            <mass value="3"/>
+            <origin rpy="0 0 0" xyz="0 0 0"/>
+            <inertia ixx="0.003" ixy = "0" ixz = "0"
+                     iyy="0.003" iyz = "0"
+                     izz="0.003" />
+        </inertial>
     <!-- caster front -->
-        <collision name="caster_front_collision">
-          <origin rpy=" 0 0 0" xyz="0.30 0 -0.05"/>
+        <collision name="caster_back_collision">
+          <origin rpy=" 0 0 0" xyz="0 0 0"/>
           <geometry>
             <sphere radius="0.05"/>
@@ -39,6 +48,43 @@
                 <mu>0</mu>
                 <mu2>0</mu2>
-                <slip1>1.0</slip1>
-                <slip2>1.0</slip2>
+                <slip1>1</slip1>
+                <slip2>1</slip2>
+              </ode>
+            </friction>
+          </surface>
+        </collision>
+        <visual name="caster_back_visual">
+          <origin rpy=" 0 0 0" xyz="0 0 0"/>
+          <geometry>
+            <sphere radius="0.05"/>
+          </geometry>
+        </visual>
+    </link>
+    <joint name="caster_back_joint" type="fixed">
+      <parent link="link_chassis"/>
+      <child link="link_caster"/>
+      <origin rpy="0 0 0" xyz="-0.25 0 -0.05"/>
+    </joint>
+    <link name="link_caster_front">
+        <inertial>
+            <mass value="1"/>
+            <origin rpy="0 0 0" xyz="0 0 0"/>
+            <inertia ixx="0.002" ixy = "0" ixz = "0"
+                     iyy="0.002" iyz = "0"
+                     izz="0.002" />
+        </inertial>
+    <!-- caster front -->
+        <collision name="caster_front_collision">
+          <origin rpy=" 0 0 0" xyz="0 0 0"/>
+          <geometry>
+            <sphere radius="0.05"/>
+          </geometry>
+          <surface>
+            <friction>
+              <ode>
+                <mu>0</mu>
+                <mu2>0</mu2>
+                <slip1>1</slip1>
+                <slip2>1</slip2>
               </ode>
             </friction>
@@ -46,5 +92,5 @@
         </collision>
         <visual name="caster_front_visual">
-          <origin rpy=" 0 0 0" xyz="0.2 0 -0.05"/>
+          <origin rpy=" 0 0 0" xyz="0 0 0"/>
           <geometry>
             <sphere radius="0.05"/>
@@ -52,36 +98,17 @@
         </visual>
     </link>
- <link name="sensor_laser">
-    <inertial>
-      <origin xyz="0 0 0" rpy="0 0 0" />
-      <mass value="1" />
-      <inertia ixx="0.001458333333" ixy="0" ixz="0"
-       iyy="0.001458333333" iyz="0"
-        izz="0.00125"/>
-    </inertial>
-    <visual>
-      <origin xyz="0 0 0" rpy="0 0 0" />
-      <geometry>
-        <cylinder radius="0.05" length="0.1"/>
-      </geometry>
-      <material name="white" />
-    </visual>
-    <collision>
-      <origin xyz="0 0 0" rpy="0 0 0"/>
-      <geometry>
-        <cylinder radius="0.05" length="0.1"/>
-      </geometry>
-    </collision>
-  </link>
-  <joint name="joint_sensor_laser" type="fixed">
-    <origin xyz="0.23 0 0.05" rpy="0 0 0"/>
-    <parent link="link_chassis"/>
-    <child link="sensor_laser"/>
-  </joint>
+    <joint name="caster_front_joint" type="fixed">
+      <parent link="link_chassis"/>
+      <child link="link_caster_front"/>
+      <origin rpy="0 0 0" xyz="0.25 0 -0.04"/>
+    </joint>
+  <!-- Create Sensor link and joint -->
+  <xacro:link_sensor name="sensor_laser" />
+  <xacro:joint_Sensor name="Sensor_joint"  child="sensor_laser" />
   <!-- Create right wheel -->
   <xacro:link_wheel name="link_right_wheel" />
-  <xacro:joint_wheel name="joint_right_wheel"  child="link_right_wheel"  origin_xyz="-0.05 0.28 0"  />
+  <xacro:joint_wheel name="joint_right_wheel"  child="link_right_wheel"  origin_xyz="0 -0.32 0"  />
 	 <!-- Create left wheel -->
   <xacro:link_wheel name="link_left_wheel" />
-  <xacro:joint_wheel name="joint_left_wheel"   child="link_left_wheel"   origin_xyz="-0.05 -0.28 0"  />
+  <xacro:joint_wheel name="joint_left_wheel"   child="link_left_wheel"   origin_xyz="0 0.32 0"  />
 </robot>
